Commit message: Added fingertips, fine visual models.

File: robots/robotiq_arg85_description.URDF (robot description, URDF)
Before this commit: robot robotiq_arg85_description, 9 links, 8 joints
Links:
- link left_inner_finger: geometry collision mesh filename=package://robotiq_arg85_description/meshes/inner_finger_coa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; visual mesh filename=package://robotiq_arg85_description/meshes/inner_finger_fin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
- link left_inner_knuckle: geometry collision mesh filename=package://robotiq_arg85_description/meshes/inner_knuckle_co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; visual mesh filename=package://robotiq_arg85_description/meshes/inner_knuckle_fi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
- link left_outer_finger: geometry collision mesh filename=package://robotiq_arg85_description/meshes/outer_finger_coa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; visual mesh filename=package://robotiq_arg85_description/meshes/outer_finger_fin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
- link left_outer_knuckle: geometry collision mesh filename=package://robotiq_arg85_description/meshes/outer_knuckle_co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; visual mesh filename=package://robotiq_arg85_description/meshes/outer_knuckle_fi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
- link right_inner_finger: geometry collision mesh filename=package://robotiq_arg85_description/meshes/inner_finger_coa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; visual mesh filename=package://robotiq_arg85_description/meshes/inner_finger_fin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
- link right_inner_knuckle: geometry collision mesh filename=package://robotiq_arg85_description/meshes/inner_knuckle_co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; visual mesh filename=package://robotiq_arg85_description/meshes/inner_knuckle_fi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
- link right_outer_finger: geometry collision mesh filename=package://robotiq_arg85_description/meshes/outer_finger_coa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; visual mesh filename=package://robotiq_arg85_description/meshes/outer_finger_fin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
- link right_outer_knuckle: geometry collision mesh filename=package://robotiq_arg85_description/meshes/outer_knuckle_co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; visual mesh filename=package://robotiq_arg85_description/meshes/outer_knuckle_fi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
Joints:
- joint left_outer_knuckle_joint: limit lower=0 upper=0.75 effort=1000 velocity=2.0 -> lower=0 upper=0.725 effort=1000 velocity=2.0

Commit message: Changed master joint name.

File: robots/robotiq_arg85_description.URDF (robot description, URDF)
Before this commit: robot robotiq_arg85_description, 9 links, 8 joints
Joints:
- removed joint left_outer_knuckle_joint
- added joint finger_joint: type revolute, parent robotiq_85_base_link, child left_outer_knuckle, origin xyz=0.0306011444260539 0 0.0627920162695395 rpy=0 0 0, axis 0 -1 0, limit lower=0 upper=0.725 effort=1000 velocity=2.0
- joint left_inner_finger_joint: mimic joint=left_outer_knuckle_joint multiplier=-1 offset=0 -> joint=finger_joint multiplier=-1 offset=0
- joint left_inner_knuckle_joint: mimic joint=left_outer_knuckle_joint multiplier=1 offset=0 -> joint=finger_joint multiplier=1 offset=0
- joint left_outer_finger_joint: mimic joint=left_outer_knuckle_joint multiplier=-1 offset=0 -> joint=finger_joint multiplier=-1 offset=0
- joint right_inner_finger_joint: mimic joint=left_outer_knuckle_joint multiplier=1 offset=0 -> joint=finger_joint multiplier=1 offset=0
- joint right_inner_knuckle_joint: mimic joint=left_outer_knuckle_joint multiplier=-1 offset=0 -> joint=finger_joint multiplier=-1 offset=0
- joint right_outer_finger_joint: mimic joint=left_outer_knuckle_joint multiplier=1 offset=0 -> joint=finger_joint multiplier=1 offset=0
- joint right_outer_knuckle_joint: mimic joint=left_outer_knuckle_joint multiplier=-1 offset=0 -> joint=finger_joint multiplier=-1 offset=0

Commit message: Removed limit and mimic properties from fixed joints.

File: robots/robotiq_arg85_description.URDF (robot description, URDF)
Before this commit: robot robotiq_arg85_description, 9 links, 8 joints
Joints:
- joint left_outer_finger_joint: limit lower=0 upper=0.8757 effort=1000 velocity=2.0 -> (none); mimic joint=finger_joint multiplier=-1 offset=0 -> (none)
- joint right_outer_finger_joint: limit lower=0 upper=0.8757 effort=1000 velocity=2.0 -> (none); mimic joint=finger_joint multiplier=1 offset=0 -> (none)
